Commit message: better two steering model

File: urdf/twosteering.xacro (robot description, xacro)
@@ -16,5 +16,5 @@
   <link name="base_link">
     <visual>
-      <origin rpy="0 ${PI/2} 0"/>
+      <origin rpy="0 ${PI/2} 0" xyz="${L/2} 0 0"/>
       <geometry>
         <cylinder length="${L}" radius="0.05"/>
@@ -65,27 +65,5 @@
 </joint>
 </xacro:macro>
- <xacro:wheel name="front" offset="${L/2}"/>
- <xacro:wheel name="rear" offset="${-L/2}"/>
-  <link name="carrot">
-      <visual>
-          <origin rpy="-1.57 0 0"/>
-          <geometry>
-              <mesh filename="package://ecn_mobile_control/urdf/carrot/carrot.dae" scale="0.003 0.003 0.003"/>
-          </geometry>
-      </visual>
-  </link>
-    <joint name="carrot_disable" type="prismatic">
-    <parent link="footprint"/>
-    <child link="carrot_disable"/>
-    <axis xyz="0 0 1"/>
-    <limit lower="-100" upper="100" velocity="10" effort="-1"/>
-  </joint>
-  <joint name="carrot" type="prismatic">
-    <parent link="carrot_disable"/>
-    <child link="carrot"/>
-    <origin xyz="0 0 0"/>
-    <axis xyz="1 0 0"/>
-    <limit lower="-100" upper="100" velocity="10" effort="-1"/>
-  </joint>
-  <link name="carrot_disable"/>
+ <xacro:wheel name="front" offset="${L}"/>
+ <xacro:wheel name="rear" offset="0"/>
 </robot>

Commit message: twosteering + costmap with footprint

File: urdf/twosteering.xacro (robot description, xacro)
@@ -2,4 +2,5 @@
 <robot name="two_steering" xmlns:xacro="http://www.ros.org/wiki/xacro">
 <xacro:property name="PI" value="3.1415926535897931"/>
+<xacro:arg name="prefix" default="robot/"/>
 <xacro:property name="radius" value=".4"/>
 <xacro:property name="L" value="1."/>
@@ -23,8 +24,8 @@
     </visual>
   </link>
-  <link name="footprint"/>
+  <link name="$(arg prefix)footprint"/>
   <joint name="footprint" type="fixed">
       <child link="base_link"/>
-      <parent link="footprint"/>
+      <parent link="$(arg prefix)footprint"/>
     <origin xyz="0 0 ${radius}"/>
    </joint>
